File: hardware/prj-kicad/cowmod-mini-fpga.sch (KiCad schematic (older format))
At the start: 10 parts, among them U2 ICE40HX1K-VQ100

Commit message: = ADD: Insert MCU and connect it to FPGA
Parts:
- added C34, C35: 100nF, cowmod-mini:SMD0603, symbol cowmod-mini:C
Connections:
- net GND: now also C34.2, C35.2
- net FMC_NWE: now reaches U2.51 (IO52)
- net FMC_NOE: now reaches U2.52 (IO53)
- net FMC_AD2: now reaches U2.53 (IO54)
- net FMC_AD3: now reaches U2.54 (IO55)
- net FMC_AD9: now reaches U2.56 (IO56)
- net FMC_AD10: now reaches U2.57 (IO57)
- net +3.3V: now reaches U2.58
- net +3.3V: now also U2.31, U2.38, U2.67, C34.1, C35.1
- net FMC_AD11: now reaches U2.59 (IO58)
- net FMC_AD12: now reaches U2.60 (IO59)
- net FMC_AD1: now reaches U2.62 (IO60_GB3)
- net FMC_CLK: now reaches U2.63 (IO61_GB2)
- net FMC_AD0: now reaches U2.64 (IO63)
- net FMC_AD15: now reaches U2.65 (IO64)
- net FMC_AD14: now reaches U2.66 (IO65)
- net FMC_AD13: now reaches U2.68 (IO67)
- net FMC_AD4: now reaches U2.69 (IO68)
- net FMC_AD5: now reaches U2.71 (IO69)
- net FMC_AD6: now reaches U2.72 (IO70)
- net FMC_AD7: now reaches U2.73 (IO71)
- net FMC_AD8: now reaches U2.74 (IO72)
- net FMC_NADV: now reaches U2.37 (IO37)
- net FMC_NE1: now reaches U2.40 (IO41)
- net FMC_WAIT: now reaches U2.41 (CBS0_IO42)
Other:
- moved on the sheet: U2B, U2C

Commit message: = ADD: Insert power supply regulators (3V3 / 1V2 / 2V5)
Connections:
- net +3.3V: now also U2.50 (VCC_SPI)
- net +2.5V: now reaches U2.75 (2V5)
- no-connect marks 21 -> 22
Changed lines of the file:
@@
 $Descr A4 11693 8268
 encoding utf-8
-Sheet 2 4
+Sheet 2 5
 Title ""
 Date ""
@@
 	1    0    0    -1
 $EndComp
+$Comp
+L cowmod-mini:+2.5V #PWR0194
+U 1 1 5E40FB1C
+P 3050 4800
+F 0 "#PWR0194" H 3050 4760 30  0001 C CNN
+F 1 "+2.5V" H 3059 4938 30  0000 C CNN
+F 2 "" H 3050 4800 60  0000 C CNN
+F 3 "" H 3050 4800 60  0000 C CNN
+	1    3050 4800
+	1    0    0    -1
+$EndComp
+Wire Wire Line
+	3050 4800 3050 4950
+$Comp
+L cowmod-mini:+3.3V #PWR0195
+U 1 1 5E42297E
+P 2850 4800
+F 0 "#PWR0195" H 2850 4760 30  0001 C CNN
+F 1 "+3.3V" H 2859 4938 30  0000 C CNN
+F 2 "" H 2850 4800 60  0000 C CNN
+F 3 "" H 2850 4800 60  0000 C CNN
+	1    2850 4800
+	1    0    0    -1
+$EndComp
+Wire Wire Line
+	2850 4800 2850 4950
+NoConn ~ 2950 4950
 $EndSCHEMATC
